File: Genesis.sch (KiCad schematic (older format))
At the start: 36 parts, among them J1 Conn_01x02_Female, J10 Conn_01x03_Female, J11 Conn_01x04_Female, J12 Conn_01x04_Female, J13 Conn_01x02_Female, J14 Conn_01x02_Female, J15 Conn_01x08_Female, J16 Conn_01x03_Female, J17 Conn_01x01_Male, J2 Jack-DC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

Commit message: Incluyo BC66 en la misma placa
Parts:
- removed D1, D2: 1N4007, Diode_THT:D_DO-41_SOD81_P10.16mm_Horizontal, symbol Diode:1N4007
- removed J1: Conn_01x02_Female, Connector_PinHeader_2.54mm:PinHeader_1x02_P2.54mm_Vertical, symbol Connector:Conn_01x02_Female
- removed J10, J16, J9: Conn_01x03_Female, Connector_JST:JST_EH_B3B-EH-A_1x03_P2.50mm_Vertical, symbol Connector:Conn_01x03_Female
- removed J11, J12: Conn_01x04_Female, Connector_JST:JST_EH_B4B-EH-A_1x04_P2.50mm_Vertical, symbol Connector:Conn_01x04_Female
- removed J13, J14: Conn_01x02_Female, TerminalBlock:TerminalBlock_bornier-2_P5.08mm, symbol Connector:Conn_01x02_Female
- removed J15, J8: Conn_01x08_Female, Connector_PinSocket_2.54mm:PinSocket_1x08_P2.54mm_Vertical, symbol Connector:Conn_01x08_Female
- removed J17, J6: Conn_01x01_Male, Connector_PinHeader_2.54mm:PinHeader_1x01_P2.54mm_Vertical, symbol Connector:Conn_01x01_Male
- removed J3, J4: Conn_01x06_Female, Connector_PinSocket_2.54mm:PinSocket_1x06_P2.54mm_Vertical, symbol Connector:Conn_01x06_Female
- removed J5: Conn_01x05_Female, Connector_JST:JST_EH_B5B-EH-A_1x05_P2.50mm_Vertical, symbol Connector:Conn_01x05_Female
- removed J7: Conn_01x03_Female, Connector_PinSocket_2.54mm:PinSocket_1x03_P2.54mm_Vertical, symbol Connector:Conn_01x03_Female
- removed R1, R3: 1k, Resistor_THT:R_Axial_DIN0207_L6.3mm_D2.5mm_P10.16mm_Horizontal, symbol Device:R
- added C5: 220n, Capacitor_SMD:C_1206_3216Metric, symbol Device:C
- added F1: Fuse, Fuse:Fuseholder_Cylinder-5x20mm_Stelvio-Kontek_PTF78_Horizontal_Open, symbol Device:Fuse
- added J1, J13, J14: Conn_01x02, TerminalBlock:TerminalBlock_bornier-2_P5.08mm, symbol Connector_Generic:Conn_01x02
- added J10, J16, J7, J9: Conn_01x03, Connector_JST:JST_EH_B3B-EH-A_1x03_P2.50mm_Vertical, symbol Connector_Generic:Conn_01x03
- added J12, J3: Conn_01x04, Connector_JST:JST_EH_B4B-EH-A_1x04_P2.50mm_Vertical, symbol Connector_Generic:Conn_01x04
- added J15, J8: Conn_01x08, Connector_PinSocket_2.54mm:PinSocket_1x08_P2.54mm_Vertical, symbol Connector_Generic:Conn_01x08
- added J17, J6: Conn_01x01, Connector_PinHeader_2.54mm:PinHeader_1x01_P2.54mm_Vertical, symbol Connector_Generic:Conn_01x01
- added J5: Conn_01x05, Connector_JST:JST_EH_B5B-EH-A_1x05_P2.50mm_Vertical, symbol Connector_Generic:Conn_01x05
- C1: value 0.33u -> 10u
- C2: value 100u -> 1u
- C3, C4: value 0.1u -> 100n; footprint Capacitor_THT:C_Disc_D3.8mm_W2.6mm_P2.50mm -> Capacitor_SMD:C_1206_3216Metric
- D3, D4: value 1N4004 -> 1N4007
- Q1, Q2: value 2N2219 -> BC547; footprint Package_TO_SOT_THT:TO-39-3 -> Package_TO_SOT_THT:TO-92
- R2, R4, R5: footprint Resistor_THT:R_Axial_DIN0207_L6.3mm_D2.5mm_P10.16mm_Horizontal -> Resistor_SMD:R_1206_3216Metric
Connections:
- net labels added: Buzzer, MISO, MOSI, PSM_EINT, PWR_KEY, RST, SCK, SS, Sensor_presencia1, Sensor_presencia2
- wire segments 114 -> 93
- no-connect marks 30 -> 20
Other:
- note added: "ARDUINO NANO"
- note added: "Bornera grande"
- note added: "Cooler"
- note added: "Power input"
- note removed: "SIM800L GSM"
- moved on the sheet: A1, C1, C2, C3, C4, D3, D4, J2, K1, K2, Q1, Q2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
